File: micromod-reset/micromod-reset.kicad_sch (KiCad schematic)
At the start: 31 parts, among them J1 Conn_01x10, SW1 DFU, SW2 nBOOT, SW3 nRST, SW4 k01, SW5 k02, SW6 k03, SW7 k04, SW8 k05, U1 74LS14, U2 74LS132, U3 74LS08

Commit message: micromod-reset, now with added test points and DRC success
Parts:
- added TP1, TP10, TP11, TP12, TP13, TP14, TP15, TP2, TP3, TP4, TP5, TP6, TP7, TP8, TP9: TestPoint_Small, TestPoint:TestPoint_Loop_D3.50mm_Drill1.4mm_Beaded, symbol Connector:TestPoint_Small
- R1: value 200k -> 10k
- R10: renamed from R11; value 200k -> 10k
- R11: renamed from R12; value 200k -> 10k
- R12: renamed from R13; value 200k -> 10k
- R13: renamed from R14; value 200k -> 10k
- R2: renamed from R4; value 200k -> 10k
- R4: renamed from R6; value 200k -> 10k
- R9: renamed from R10; value 200k -> 10k
- renumbered C3 to C2, C4 to C3, C2 to C4, R5 to R3, R8 to R5, R2 to R6, R3 to R7, R9 to R8
Connections:
- net ~{k13} is gone; now on net ~{k03}: U1.6, U3.4
- net +3V3: now also TP15.1
- net GND: now also TP14.1
- net ~{k03}: now also TP3.1; no longer U1.2, U3.1
- net OSC_OUT: now reaches R5.1, R6.1, R7.1, U2.10, U2.6, U2.9
- net OSC_OUT: now also TP11.1
- net OSC_RC: now reaches C4.1, R5.2, R6.2, R7.2, R8.2, U2.5
- net OSC_RC: now also TP12.1
- net ~{OSC_OUT}: now reaches U2.12, U2.13, U2.8
- net ~{OSC_OUT}: now also TP13.1
- net ~{k01}&&~{k02}&&~{k03}&&~{k04}&&~{k05}: now reaches D1.2 (A), R2.2, SW1.2, U2.4, U3.11
- net ~{k01}&&~{k02}&&~{k03}&&~{k04}&&~{k05}: now also TP9.1
- net BOOT_RC: now reaches C1.1, D1.1 (K), R3.2, U2.1, U2.2
- net BOOT_RC: now also TP10.1
- net ~{k03}&&~{k07} renamed ~{k01}&&~{k02}
- net ~{k01}&&~{k02}: now also TP7.1
- net ~{k07} renamed ~{k02}
- net ~{k02}: now also TP2.1
- net ~{k13}&&~{k17} renamed ~{k03}&&~{k04}
- net ~{k03}&&~{k04}: now also TP6.1
- net ~{k13}&&~{k17}&&~{k23} renamed ~{k03}&&~{k04}&&~{k05}
- net ~{k03}&&~{k04}&&~{k05}: now also TP8.1
- net ~{k17} renamed ~{k04}
- net ~{k04}: now also TP4.1
- net ~{k23} renamed ~{k05}
- net ~{k05}: now also TP5.1
- new net ~{k01}: TP1.1, U1.2, U3.1
Other:
- moved on the sheet: R4, R8, SW3, U1F, U2D

Commit message: Updated JLC to match fixed circuit.
Parts:
- R1, R10, R11, R12, R13, R2, R4, R9: value 10k -> 200k
Changed lines of the file:
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@@
 			)
 		)
-		(property "Value" "10k"
+		(property "Value" "200k"
 			(at 50.8 152.4 0)
 			(effects
@@
 			)
 		)
-		(property "Value" "10k"
+		(property "Value" "200k"
 			(at 33.02 152.4 0)
 			(effects
@@
 			)
 		)
-		(property "Value" "10k"
+		(property "Value" "200k"
 			(at 151.13 45.72 0)
 			(effects
@@
 			)
 		)
-		(property "Value" "10k"
+		(property "Value" "200k"
 			(at 59.69 152.4 0)
 			(effects
@@
 			)
 		)
-		(property "Value" "10k"
+		(property "Value" "200k"
 			(at 262.89 60.96 0)
 			(effects
@@
 			)
 		)
-		(property "Value" "10k"
+		(property "Value" "200k"
 			(at 68.58 152.4 0)
 			(effects
@@
 			)
 		)
-		(property "Value" "10k"
+		(property "Value" "200k"
 			(at 222.25 31.75 0)
 			(effects
@@
 			)
 		)
-		(property "Value" "10k"
+		(property "Value" "200k"
 			(at 41.91 152.4 0)
 			(effects
